Commit message: maaran 4 fixed

File: rover_desc/urdf/robot_4.urdf.xacro (robot description, xacro)
@@ -2,56 +2,6 @@
 <robot xmlns:xacro="http://www.ros.org/wiki/xacro" name="robo4">
     <xacro:include filename="$(find rover_desc)/urdf/inertial_macros.xacro"/>
+    <xacro:include filename="$(find rover_desc)/urdf/gazebo_control4.xacro"/>
     <xacro:property name="robot_namespace" value="robot4" />
-    <gazebo>
-        <plugin name="gazebo_control" filename="libgazebo_ros_diff_drive.so">
-            <num_wheel_pairs>2</num_wheel_pairs>
-            <ros>
-                <namespace>${robot_namespace}</namespace>
-            </ros>
-            <left_joint>lb_wheel_joint</left_joint>
-            <right_joint>rb_wheel_joint</right_joint>
-            <left_joint>lf_wheel_joint</left_joint>
-            <right_joint>rf_wheel_joint</right_joint>
-            <wheel_separation>1.2</wheel_separation>
-            <wheel_diameter>0.45</wheel_diameter>
-            <command_topic>cmd_vel</command_topic>
-            <update_rate>50</update_rate>
-            <max_wheel_torque>100</max_wheel_torque>
-            <max_wheel_acceleration>5.0</max_wheel_acceleration>
-            <odometry_frame>odom</odometry_frame>
-            <robot_base_frame>base_link</robot_base_frame>
-            <publish_odom>true</publish_odom>
-            <publish_odom_tf>true</publish_odom_tf>
-            <publish_wheel_tf>true</publish_wheel_tf>
-        </plugin>
-    </gazebo>
-    <gazebo reference="lb_wheel">
-        <mu1>0.5</mu1>
-        <mu2>0.5</mu2>
-    </gazebo>
-    <gazebo reference="lf_wheel">
-        <mu1>0.5</mu1>
-        <mu2>0.5</mu2>
-    </gazebo>
-    <gazebo reference="rb_wheel">
-        <mu1>0.5</mu1>
-        <mu2>0.5</mu2>
-    </gazebo>
-    <gazebo reference="rf_wheel">
-        <mu1>0.5</mu1>
-        <mu2>0.5</mu2>
-    </gazebo>
-    <material name="white">
-        <color rgba="1 1 1 1" />
-    </material>
-    <material name="orange">
-        <color rgba="1 0.3 0.1 1"/>
-    </material>
-    <material name="blue">
-        <color rgba="0.2 0.2 1 1"/>
-    </material>
-    <material name="black">
-        <color rgba="0 0 0 1"/>
-    </material>
     <link name="base_link">
         <visual>
